File: hw/mcu.kicad_sch (KiCad schematic)
At the start: 31 parts, among them J3 USB_C_Receptacle_USB2.0_14P, J4 Conn_01x06, U1 AP2112K-3.3, U2 ESP32-C3-12F

Commit message: Fix included libraries. Arrange schematic notes. Add mechanical parts to schematic.
Parts:
- added KN1: 20 mm, symbol Mechanical:Mechanical_Shape
Other:
- moved on the sheet: C10, C9, JP2, R11, R12, R13, R14, R15, SW1, SW2, U2
