File: hw/pwr.kicad_sch (KiCad schematic)
At the start: 15 parts, among them J1 Screw_Terminal_01x02, K1 Relay_DPDT, Q8 MMBT3904

Commit message: Update design
Parts:
- removed TP1: 3V3, TestPoint:TestPoint_Pad_D1.0mm, symbol Connector:TestPoint_Flag
- added J2: Conn_01x02_Pin, Connector_PinSocket_2.54mm:PinSocket_1x02_P2.54mm_Vertical, symbol Connector:Conn_01x02_Pin
- added JP1: SolderJumper_2_Bridged, Jumper:SolderJumper-2_P1.3mm_Bridged_RoundedPad1.0x1.5mm, symbol Jumper:SolderJumper_2_Bridged
- R1: value 120 -> 330
- renumbered Q8 to Q1, TP2 to TP1
Connections:
- net +3V3: now also J2.2 (Pin_2), JP1.2 (B); no longer A1.4 (+Vout), C2.1
- new net: A1.4 (+Vout), C2.1, J2.1 (Pin_1), JP1.1 (A)
Other:
- title: LEDDs -> Power
- moved on the sheet: A1, C1, C2, C3, D1, D2, J1, K1, Q1, R1, R2, RV1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
